File: connectors.kicad_sch (KiCad schematic)
At the start: 10 parts, among them CN102 Expansion, CN105 JOY1, CN202 HuCARD

Commit message: Add contact info the schematics for publishing.
Other:
- company: (none) -> By Cosam
Changed lines of the file:
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@@
   (title_block
     (title "PC Engine Connectors")
-    (date "2023-09-20")
-    (rev "1.2")
-    (comment 1 "Differences reverse engineered from original PWD-623A board")
-    (comment 2 "Adapted from existing TurboGrafx-16 schematics by Cosam")
+    (date "2023-11-15")
+    (rev "1.2.1")
+    (company "By Cosam")
+    (comment 1 "https://github.com/Board-Folk/PC-Engine")
+    (comment 2 "For contributions or corrections please visit:")
+    (comment 3 "Differences reverse engineered from original PWD-623A board")
+    (comment 4 "Adapted from existing TurboGrafx-16 schematics")
   )
   (junction (at 313.69 119.38) (diameter 0) (color 0 0 0 0)
